File: PCB/PCB.kicad_pcb (KiCad board)
At the start: 2 copper layers, 22 x 22 mm, 4 parts

Commit message: kill me
Parts:
- removed REF** (x4): HTSSOP-16-1EP_4.4x5mm_P0.65mm_EP3.4x5mm_Mask2.46x2.31mm_The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, Package_SO:HTSSOP-16-1EP_4.4x5mm_P0.65mm_EP3.4x5mm_Mask2.46x2.31mm_ThermalVias
- added C1: 22nf, Capacitor_SMD:C_0402_1005Metric, F.Cu at (103.3, 98.0)
- added C3: 100nf, Capacitor_SMD:C_0402_1005Metric, F.Cu at (104.7, 95.9)
- added C4: 100nf, Capacitor_SMD:C_0402_1005Metric, F.Cu at (105.7, 96.9)
- added D1: LED, LED_SMD:LED_0805_2012Metric, F.Cu at (108.5, 108.4)
- added J1: GPIO/Control, Connector_PinHeader_1.00mm:PinHeader_1x06_P1.00mm_Vertical, F.Cu at (101.4, 111.0)
- added J2: POWER, Taranium-libs:3P_Screw_Terminal, B.Cu at (97.0, 99.0)
- added R2: 1k, Capacitor_SMD:C_0402_1005Metric, F.Cu at (104.3, 107.9)
- added R4: 10k, Capacitor_SMD:C_0402_1005Metric, F.Cu at (103.3, 108.2)
- added R5: 2k, Capacitor_SMD:C_0402_1005Metric, F.Cu at (105.9, 108.3)
- added U1: ~, Package_SO:HTSSOP-16-1EP_4.4x5mm_P0.65mm_EP3.4x5mm_Mask2.46x2.31mm_ThermalVias, F.Cu at (104.4, 102.9)
- added U2: ~, Package_TO_SOT_SMD:SOT-353_SC-70-5, F.Cu at (99.8, 106.8)
Routing:
- net +3V3: track 0.00 -> 17.3 mm, vias 0 -> 2
- net /SLEEP: track 0.00 -> 10.6 mm, vias 0 -> 2
- net /IO2: track 0.00 -> 7.02 mm
- net GND: track 0.00 -> 6.48 mm, vias 0 -> 5
- net Net-(D1-A): track 0.00 -> 4.58 mm, vias 0 -> 2
- net /IO1: track 0.00 -> 3.61 mm
- net Net-(U1-VREF): track 0.00 -> 2.55 mm
- net Net-(U1-nFAULT): track 0.00 -> 1.76 mm
- net Net-(U1-CPL): track 0.00 -> 1.60 mm
Other:
- board outline removed

Commit message: slime dookie
Parts:
- moved C3 0.10 mm to (104.7, 95.8)
Routing:
- net +24V: track 0.00 -> 4.74 mm
- net Net-(U1-VCP): track 0.00 -> 4.34 mm
- net Net-(U1-CPH): track 0.00 -> 2.83 mm
- net GND: track 6.48 -> 7.92 mm, vias 5 -> 6
- added copper zone on F.Cu, net +24V
- added copper zone on B.Cu, net GND
Changed lines of the file:
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@@
 	)
 	(setup
+		(stackup
+			(layer "F.SilkS"
+				(type "Top Silk Screen")
+			)
+			(layer "F.Paste"
+				(type "Top Solder Paste")
+			)
+			(layer "F.Mask"
+				(type "Top Solder Mask")
+				(thickness 0.01)
+			)
+			(layer "F.Cu"
+				(type "copper")
+				(thickness 0.035)
+			)
+			(layer "dielectric 1"
+				(type "core")
+				(thickness 1.51)
+				(material "FR4")
+				(epsilon_r 4.5)
+				(loss_tangent 0.02)
+			)
+			(layer "B.Cu"
+				(type "copper")
+				(thickness 0.035)
+			)
+			(layer "B.Mask"
+				(type "Bottom Solder Mask")
+				(thickness 0.01)
+			)
+			(layer "B.Paste"
+				(type "Bottom Solder Paste")
+			)
+			(layer "B.SilkS"
+				(type "Bottom Silk Screen")
+			)
+			(copper_finish "None")
+			(dielectric_constraints no)
+		)
 		(pad_to_mask_clearance 0)
 		(allow_soldermask_bridges_in_footprints no)
@@
 		(capping no)
 		(filling no)
+		(zone_defaults)
 		(pcbplotparams
 			(layerselection 0x00000000_00000000_55555555_5755f5ff)
@@
 	(footprint "Capacitor_SMD:C_0402_1005Metric"
 		(layer "F.Cu")
-		(at 104.7 95.9)
+		(at 104.7 95.8)
 		(descr "Capacitor SMD 0402 (1005 Metric), square (rectangular) end terminal, IPC-7351 nominal, (Body size source: IPC-SM-782 page 76, https://www.pcb-3d.com/wordpress/wp-content/uploads/ipc-sm-782a_amendment_1_and_2.pdf)")
 		(tags "capacitor")
@@
 		(stroke
 			(width 0.1)
-			(type default)
+			(type solid)
 		)
 		(fill no)
-		(layer "F.SilkS")
+		(layer "Dwgs.User")
+	)
+	(segment
+		(start 104.06 100.0375)
+		(end 104.06 98.28)
+		(width 0.2)
+		(layer "F.Cu")
+		(net "Net-(U1-CPH)")
+	)
+	(segment
+		(start 104.06 98.28)
+		(end 103.3 97.52)
+		(width 0.2)
+		(layer "F.Cu")
+		(net "Net-(U1-CPH)")
 	)
 	(segment
@@
 	)
 	(segment
+		(start 104.71 98.364314)
+		(end 104.22 97.874314)
+		(width 0.2)
+		(layer "F.Cu")
+		(net "Net-(U1-VCP)")
+	)
+	(segment
+		(start 104.71 100.0375)
+		(end 104.71 98.364314)
+		(width 0.2)
+		(layer "F.Cu")
+		(net "Net-(U1-VCP)")
+	)
+	(segment
+		(start 104.22 97.874314)
+		(end 104.22 95.9)
+		(width 0.2)
+		(layer "F.Cu")
+		(net "Net-(U1-VCP)")
+	)
+	(segment
+		(start 105.4 99.936593)
+		(end 105.4 98.263407)
+		(width 0.2)
+		(layer "F.Cu")
+		(net "+24V")
+	)
+	(segment
+		(start 105.3 96.98)
+		(end 105.22 96.9)
+		(width 0.2)
+		(layer "F.Cu")
+		(net "+24V")
+	)
+	(segment
+		(start 105.3 99.936593)
+		(end 105.3 96.98)
+		(width 0.2)
+		(layer "F.Cu")
+		(net "+24V")
+	)
+	(segment
 		(start 105.36 105.7625)
 		(end 106.01 105.7625)
@@
 	(segment
 		(start 102.11 100.0375)
-		(end 101.4625 100.0375)
-		(width 0.2)
+		(end 102.71 100.0375)
+		(width 0.6)
 		(layer "F.Cu")
 		(net "GND")
 	)
 	(segment
-		(start 106.66 100.0375)
-		(end 107.4375 100.0375)
-		(width 0.2)
-		(layer "F.Cu")
-		(net "GND")
-	)
-	(segment
-		(start 107.4375 100.0375)
-		(end 107.5 100.1)
-		(width 0.2)
+		(start 101.3375 100.0375)
+		(end 101.3 100)
+		(width 0.6)
 		(layer "F.Cu")
 		(net "GND")
@@
 	)
 	(segment
-		(start 102.76 100.0375)
-		(end 102.11 100.0375)
-		(width 0.2)
+		(start 106.18 96.9)
+		(end 107.2 96.9)
+		(width 0.6)
 		(layer "F.Cu")
 		(net "GND")
@@
 	)
 	(segment
-		(start 101.4625 100.0375)
-		(end 101.4 100.1)
-		(width 0.2)
+		(start 106.71 100.0875)
+		(end 106.71 100.0375)
+		(width 0.6)
 		(layer "F.Cu")
 		(net "GND")
@@
 	)
 	(segment
+		(start 107.9 100.1)
+		(end 106.7225 100.1)
+		(width 0.6)
+		(layer "F.Cu")
+		(net "GND")
+	)
+	(segment
+		(start 106.7225 100.1)
+		(end 106.71 100.0875)
+		(width 0.6)
+		(layer "F.Cu")
+		(net "GND")
+	)
+	(segment
+		(start 102.11 100.0375)
+		(end 101.3375 100.0375)
+		(width 0.6)
+		(layer "F.Cu")
+		(net "GND")
+	)
+	(segment
 		(start 100.6375 106.8)
 		(end 100.6375 106.15)
@@
 	)
 	(via
-		(at 101.4 100.1)
-		(size 0.6)
-		(drill 0.3)
+		(at 101.3 100)
+		(size 0.8)
+		(drill 0.4)
 		(layers "F.Cu" "B.Cu")
 		(net "GND")
@@
 	)
 	(via
-		(at 107.5 100.1)
+		(at 108.5 110.4)
 		(size 0.6)
 		(drill 0.3)
@@
 	)
 	(via
-		(at 108.5 110.4)
+		(at 107.9 100.1)
 		(size 0.6)
 		(drill 0.3)
 		(layers "F.Cu" "B.Cu")
+		(free yes)
 		(net "GND")
 	)
@@
 		(net "GND")
 	)
+	(via
+		(at 107.2 96.9)
+		(size 0.8)
+		(drill 0.4)
+		(layers "F.Cu" "B.Cu")
+		(net "GND")
+	)
 	(segment
 		(start 104.3 108.38)
@@
 		(net "/IO1")
 	)
+	(zone
+		(net "+24V")
+		(layer "F.Cu")
+		(hatch edge 0.5)
+		(connect_pads
+			(clearance 0.5)
+		)
+		(min_thickness 0.25)
+		(fill yes
+			(thermal_gap 0.5)
+			(thermal_bridge_width 0.5)
+			(island_removal_mode 0)
+		)
+		(polygon
+			(pts
+				(xy 90.9 92.7) (xy 88.9 114) (xy 117.2 114.7) (xy 116.5 92.5) (xy 106.9 91.4)
+			)
+		)
+	)
+	(zone
+		(net "GND")
+		(layer "B.Cu")
+		(hatch edge 0.5)
+		(priority 1)
+		(connect_pads
+			(clearance 0.5)
+		)
+		(min_thickness 0.25)
+		(fill yes
+			(thermal_gap 0.5)
+			(thermal_bridge_width 0.5)
+			(island_removal_mode 0)
+		)
+		(polygon
+			(pts
+				(xy 89.9 91) (xy 85.6 116.5) (xy 118.8 116.2) (xy 119.6 88.7)
+			)
+		)
+	)
 	(embedded_fonts no)

Commit message: commite
Parts:
- added C2: 22uf, Capacitor_THT:CP_Radial_D10.0mm_P5.00mm, B.Cu at (108.8, 96.8)
- added J3: OUTPUT2, Taranium-libs:Electromagnet Power Output, F.Cu at (111.2, 96.6)
- added J4: OUTPUT1, Taranium-libs:Electromagnet Power Output, F.Cu at (97.6, 110.5)
- J1: footprint Connector_PinHeader_1.00mm:PinHeader_1x06_P1.00mm_Vertical -> Connector_PinHeader_1.00mm:PinHeader_1x05_P1.00mm_Vertical; moved to B.Cu
- moved J2 1.00 mm to (98.0, 99.0)
- turned J1 to -90 degrees
Routing:
- net /OUT2: track 0.00 -> 6.76 mm
- net +24V: track 4.74 -> 8.71 mm
- net +3V3: track 17.3 -> 16.1 mm
- removed copper zone on F.Cu, net +24V
- removed copper zone on B.Cu, net GND
Other:
- board outline added: 17 x 17 mm

Commit message: bleh
Parts:
- added C1: 22nf, Capacitor_SMD:C_0402_1005Metric, F.Cu at (154.3, 98.0)
- added C1: 22nf, Capacitor_SMD:C_0402_1005Metric, F.Cu at (137.3, 98.0)
- added C2: 22uf, Capacitor_THT:CP_Radial_D10.0mm_P5.00mm, B.Cu at (142.8, 96.8)
- added C2: 22uf, Capacitor_THT:CP_Radial_D10.0mm_P5.00mm, B.Cu at (159.8, 96.8)
- added C3: 100nf, Capacitor_SMD:C_0402_1005Metric, F.Cu at (155.7, 95.8)
- added C3: 100nf, Capacitor_SMD:C_0402_1005Metric, F.Cu at (138.7, 95.8)
- added C4: 100nf, Capacitor_SMD:C_0402_1005Metric, F.Cu at (139.7, 96.9)
- added C4: 100nf, Capacitor_SMD:C_0402_1005Metric, F.Cu at (156.7, 96.9)
- added C5: 22nf, Capacitor_SMD:C_0402_1005Metric, F.Cu at (120.3, 98.0)
- added C6: 100nf, Capacitor_SMD:C_0402_1005Metric, F.Cu at (121.7, 95.8)
- added C7: 100nf, Capacitor_SMD:C_0402_1005Metric, F.Cu at (122.7, 96.9)
- added C8: 22uf, Capacitor_THT:CP_Radial_D10.0mm_P5.00mm, B.Cu at (125.8, 96.8)
- added D1: LED, LED_SMD:LED_0805_2012Metric, F.Cu at (142.5, 108.4)
- added D1: LED, LED_SMD:LED_0805_2012Metric, F.Cu at (159.5, 108.4)
- added D2: LED, LED_SMD:LED_0805_2012Metric, F.Cu at (125.5, 108.4)
- added J3: OUTPUT2, Taranium-libs:Electromagnet Power Output, F.Cu at (145.2, 96.6)
- added J3: OUTPUT2, Taranium-libs:Electromagnet Power Output, F.Cu at (162.2, 96.6)
- added J4: OUTPUT1, Taranium-libs:Electromagnet Power Output, F.Cu at (131.5, 110.5)
- added J4: OUTPUT1, Taranium-libs:Electromagnet Power Output, F.Cu at (148.5, 110.5)
- added J5: OUTPUT2, Taranium-libs:Electromagnet Power Output, F.Cu at (128.2, 96.6)
- added J6: OUTPUT1, Taranium-libs:Electromagnet Power Output, F.Cu at (114.5, 110.5)
- added R2: 1k, Capacitor_SMD:C_0402_1005Metric, F.Cu at (155.3, 107.9)
- added R2: 1k, Capacitor_SMD:C_0402_1005Metric, F.Cu at (138.3, 107.9)
- added R3: 1k, Capacitor_SMD:C_0402_1005Metric, F.Cu at (121.3, 107.9)
- added R4: 10k, Capacitor_SMD:C_0402_1005Metric, F.Cu at (154.3, 108.2)
- added R4: 10k, Capacitor_SMD:C_0402_1005Metric, F.Cu at (137.3, 108.2)
- added R5: 2k, Capacitor_SMD:C_0402_1005Metric, F.Cu at (139.9, 108.3)
- added R5: 2k, Capacitor_SMD:C_0402_1005Metric, F.Cu at (156.9, 108.3)
- added R6: 10k, Capacitor_SMD:C_0402_1005Metric, F.Cu at (120.3, 108.2)
- added R7: 2k, Capacitor_SMD:C_0402_1005Metric, F.Cu at (122.9, 108.3)
- added U1: ~, Package_SO:HTSSOP-16-1EP_4.4x5mm_P0.65mm_EP3.4x5mm_Mask2.46x2.31mm_ThermalVias, F.Cu at (155.4, 102.9)
- added U1: ~, Package_SO:HTSSOP-16-1EP_4.4x5mm_P0.65mm_EP3.4x5mm_Mask2.46x2.31mm_ThermalVias, F.Cu at (138.4, 102.9)
- added U2: ~, Package_TO_SOT_SMD:SOT-353_SC-70-5, F.Cu at (151.0, 106.8)
- added U2: ~, Package_TO_SOT_SMD:SOT-353_SC-70-5, F.Cu at (134.0, 106.8)
- added U3: ~, Package_TO_SOT_SMD:SOT-353_SC-70-5, F.Cu at (117.0, 106.8)
- added U4: ~, Package_SO:HTSSOP-16-1EP_4.4x5mm_P0.65mm_EP3.4x5mm_Mask2.46x2.31mm_ThermalVias, F.Cu at (121.4, 102.9)
- moved J1 17.0 mm to (118.4, 111.0)
- moved U2 0.20 mm to (100.0, 106.8)
- moved J4 0.14 mm to (97.5, 110.5)
Routing:
- net +3V3: track 16.1 -> 96.6 mm, vias 2 -> 8
- net /IO2: track 7.02 -> 83.8 mm, vias 0 -> 2
- net /SLEEP: track 10.6 -> 72.2 mm, vias 2 -> 5
- net /OUT1: track 0.00 -> 54.5 mm, vias 0 -> 8
- net +24V: track 8.71 -> 46.6 mm
- net GND: track 7.92 -> 31.6 mm, vias 6 -> 24
- net /OUT2: track 6.76 -> 27.0 mm
- net Net-(D1-A): track 4.58 -> 18.7 mm, vias 2 -> 8
- net /IO1: track 3.61 -> 17.2 mm
- net Net-(U1-VCP): track 4.34 -> 17.4 mm
- net Net-(U1-CPH): track 2.83 -> 11.3 mm
- net Net-(U1-VREF): track 2.55 -> 10.2 mm
- net Net-(U1-nFAULT): track 1.76 -> 7.03 mm
- net Net-(U1-CPL): track 1.60 -> 6.41 mm
Other:
- board size 17 x 17 mm -> 68 x 17 mm

Commit message: bleh
Parts:
- moved C6 1.56 mm to (120.7, 97.0)
- moved C10 1.51 mm to (137.7, 96.9)
- moved C3 1.51 mm to (103.7, 96.9)
- moved C14 1.47 mm to (154.7, 96.9)
- moved C5 0.50 mm to (120.3, 98.5), turned to 0 degrees
- moved C1 0.47 mm to (103.4, 98.5), turned to 0 degrees
- moved C13 0.45 mm to (154.3, 98.5), turned to 0 degrees
- moved C9 0.41 mm to (137.4, 98.4), turned to 0 degrees
- renumbered C3 to C10, C4 to C11, C2 to C12, C1 to C13, C3 to C14, C4 to C15, C2 to C16, C1 to C9, D1 to D3, D1 to D4, J4 to J10, J3 to J7, J4 to J8, J3 to J9, R5 to R10, R2 to R11, R4 to R12, R5 to R13, R2 to R8, R4 to R9, U2 to U5, U1 to U6, U2 to U7, U1 to U8
Connections:
- J1 pad 2: unconnected-(J1-Pin_2-Pad2) -> /IO3
- J1 pad 3: unconnected-(J1-Pin_3-Pad3) -> /IO4
- J1 pad 4: unconnected-(J1-Pin_4-Pad4) -> /IO5
- U3 pad 1: /IO2 -> /IO3
- U4 pad 2: /IO2 -> /IO3
- U5 pad 1: /IO2 -> /IO4
- U6 pad 2: /IO2 -> /IO4
- U7 pad 1: /IO2 -> /IO5
- U8 pad 2: /IO2 -> /IO5
Routing:
- net GND: track 31.6 -> 169.8 mm, vias 24 -> 27
- net /IO2: track 83.8 -> 22.7 mm, vias 2 -> 0
- net /IO5: track 0.00 -> 38.9 mm, vias 0 -> 1
- net /IO4: track 0.00 -> 22.5 mm, vias 0 -> 1
- net /IO3: track 0.00 -> 7.48 mm
- net Net-(U1-CPH): track 11.3 -> 6.74 mm
- net Net-(U1-VCP): track 17.4 -> 15.1 mm
- net +3V3: track 96.6 -> 98.5 mm
- net +24V: track 46.6 -> 45.0 mm, vias 0 -> 2
- net /OUT1: track 54.5 -> 53.3 mm
- net Net-(U1-CPL): track 6.41 -> 7.26 mm
- added copper zone on B.Cu, net +24V
- added copper zone on F.Cu, net GND
Other:
- outline, holes or cut-outs redrawn

Commit message: guh
Parts:
- added H1: MountingHole, MountingHole:MountingHole_2.2mm_M2_Pad_Via, F.Cu at (161.4, 109.4)
- added H2: MountingHole, MountingHole:MountingHole_2.2mm_M2_Pad_Via, F.Cu at (115.8, 102.1)
- moved D4 4.26 mm to (155.9, 110.8), turned to 0 degrees
- moved D3 0.58 mm to (142.2, 108.9)
Routing:
- net GND: track 169.8 -> 155.2 mm, vias 27 -> 25
- net /OUT1: track 53.3 -> 54.0 mm

Commit message: potato
Parts:
- C12, C16, C2, C8: footprint Capacitor_THT:CP_Radial_D10.0mm_P5.00mm -> Capacitor_THT:CP_Radial_D5.0mm_P2.00mm
- moved C8 8.68 mm to (117.1, 97.0)
- moved C16 8.60 mm to (151.2, 96.8)
- moved C12 8.35 mm to (134.4, 96.9)
- moved C2 2.66 mm to (106.2, 96.2), turned to 0 degrees
- moved J2 2.62 mm to (98.5, 101.6)
- moved H2 1.23 mm to (114.8, 102.8)
- moved C4 1.01 mm to (106.0, 97.9)
- moved C7 0.67 mm to (122.9, 97.5)
Routing:
- net +3V3: track 98.5 -> 88.3 mm
- net GND: track 155.2 -> 163.7 mm, vias 25 -> 27
- net +24V: track 45.0 -> 41.6 mm
- net /OUT1: track 54.0 -> 51.4 mm
- net Net-(D1-A): track 18.6 -> 19.8 mm

Commit message: commit
Connections:
- C2 pad 1: +24V -> +12V
- C3 pad 2: +24V -> +12V
- C4 pad 2: +24V -> +12V
- J2 pad 3: +24V -> +12V
- U1 pad 11: +24V -> +12V
Routing:
- net +12V: track 0.00 -> 11.3 mm, vias 0 -> 2
- net +24V: track 41.6 -> 30.3 mm, vias 2 -> 0
- net +3V3: track 88.3 -> 91.8 mm
- net GND: track 163.7 -> 161.2 mm
- added copper zone on B.Cu, net +12V
- removed copper zone on B.Cu, net +24V
