File: PCB/PCB.kicad_sch (KiCad schematic)
At the start: 11 parts, among them J1 GPIO/Control, J2 POWER

Commit message: kill me
Parts:
- removed R1: 4.8k, symbol Device:R_Small
- removed R3: 1k, symbol Device:R_Small
- removed U2: (no value), symbol Taranium-libs:74LVC1G74
- added D1: LED, LED_SMD:LED_0805_2012Metric, symbol Device:LED
- added R4: 10k, Capacitor_SMD:C_0402_1005Metric, symbol Device:R_Small
- added R5: 2k, Capacitor_SMD:C_0402_1005Metric, symbol Device:R_Small
- added U2: (no value), Package_TO_SOT_SMD:SOT-353_SC-70-5, symbol Taranium-libs:SN74LVC1G02
- C1, C3, C4: footprint (none) -> Capacitor_SMD:C_0402_1005Metric
- J1: footprint (none) -> Connector_PinHeader_1.00mm:PinHeader_1x06_P1.00mm_Vertical
- J2: footprint (none) -> Taranium-libs:3P_Screw_Terminal
- R2: value 10k -> 1k; footprint (none) -> Capacitor_SMD:C_0402_1005Metric
Connections:
- net D1 is gone; now on net IO2: J1.1 (Pin_1)
- net +24V: now also J2.3 (Pin_3); no longer J2.1 (Pin_1)
- net +3V3: now also J2.1 (Pin_1), R4.2, R5.1, U2.5 (VCC); no longer J2.3 (Pin_3), R2.1
- net GND: now also U1.6 (IPROPI), D1.1 (K), U2.2 (B), U2.3 (GND)
- net IO1: now also U2.4 (Y)
- net IO2: now also U2.1 (A)
- net SLEEP: now also R4.1
- net VREF: no longer names the net of U1.5 (VREF)
- net VREF: now also R5.2
- new net: D1.2 (A), R2.1
Other:
- moved on the sheet: R2

Commit message: slime dookie
Parts:
- added J3: OUTPUT2, symbol Connector:Conn_01x01_Pin
- added J4: OUTPUT1, symbol Connector:Conn_01x01_Pin
Connections:
- net OUT1: now also J4.1 (Pin_1)
- net OUT2: now also J3.1 (Pin_1)
Changed lines of the file:
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@@
+		)
+	)
+	(label "OUT2"
+		(at 132.08 73.66 0)
+		(effects
+			(font
+				(size 1.27 1.27)
+			)
+			(justify left bottom)
 		)
 	)
@@
 		)
 	)
+	(label "OUT1"
+		(at 133.35 81.28 0)
+		(effects
+			(font
+				(size 1.27 1.27)
+			)
+			(justify left bottom)
+		)
+	)
 	(label "OUT2"
 		(at 104.14 92.71 0)
@@
 	)
 	(symbol
+		(lib_id "Connector:Conn_01x01_Pin")
+		(at 128.27 81.28 0)
+		(unit 1)
+		(body_style 1)
+		(exclude_from_sim no)
+		(in_bom yes)
+		(on_board yes)
+		(in_pos_files yes)
+		(dnp no)
+		(fields_autoplaced yes)
+		(property "Reference" "J4"
+			(at 128.905 76.2 0)
+			(show_name no)
+			(do_not_autoplace no)
+			(effects
+				(font
+					(size 1.27 1.27)
+				)
+			)
+		)
+		(property "Value" "OUTPUT1"
+			(at 128.905 78.74 0)
+			(show_name no)
+			(do_not_autoplace no)
+			(effects
+				(font
+					(size 1.27 1.27)
+				)
+			)
+		)
+		(property "Footprint" ""
+			(at 128.27 81.28 0)
+			(hide yes)
+			(show_name no)
+			(do_not_autoplace no)
+			(effects
+				(font
+					(size 1.27 1.27)
+				)
+			)
+		)
+		(property "Datasheet" ""
+			(at 128.27 81.28 0)
+			(hide yes)
+			(show_name no)
+			(do_not_autoplace no)
+			(effects
+				(font
+					(size 1.27 1.27)
+				)
+			)
+		)
+		(property "Description" "Generic connector, single row, 01x01, script generated"
+			(at 128.27 81.28 0)
+			(hide yes)
+			(show_name no)
+			(do_not_autoplace no)
+			(effects
+				(font
+					(size 1.27 1.27)
+				)
+			)
+		)
+		(pin "1"
+		)
+		(instances
+			(project "PCB"
+				(path "/cdb7748a-e4ea-465a-80fd-c707816a3e95"
+					(reference "J4")
+					(unit 1)
+				)
+			)
+		)
+	)
+	(symbol
 		(lib_id "power:GND")
 		(at 118.11 95.25 0)
@@
 					(unit 1)
 				)
+			)
+		)
+	)
+	(symbol
+		(lib_id "Connector:Conn_01x01_Pin")
+		(at 127 73.66 0)
+		(unit 1)
+		(body_style 1)
+		(exclude_from_sim no)
+		(in_bom yes)
+		(on_board yes)
+		(in_pos_files yes)
+		(dnp no)
+		(fields_autoplaced yes)
+		(property "Reference" "J3"
+			(at 127.635 68.58 0)
+			(show_name no)
+			(do_not_autoplace no)
+			(effects
+				(font
+					(size 1.27 1.27)
+				)
+			)
+		)
+		(property "Value" "OUTPUT2"
+			(at 127.635 71.12 0)
+			(show_name no)
+			(do_not_autoplace no)
+			(effects
+				(font
+					(size 1.27 1.27)
+				)
+			)
+		)
+		(property "Footprint" ""
+			(at 127 73.66 0)
+			(hide yes)
+			(show_name no)
+			(do_not_autoplace no)
+			(effects
+				(font
+					(size 1.27 1.27)
+				)
+			)
+		)
+		(property "Datasheet" ""
+			(at 127 73.66 0)
+			(hide yes)
+			(show_name no)
+			(do_not_autoplace no)
+			(effects
+				(font
+					(size 1.27 1.27)
+				)
+			)
+		)
+		(property "Description" "Generic connector, single row, 01x01, script generated"
+			(at 127 73.66 0)
+			(hide yes)
+			(show_name no)
+			(do_not_autoplace no)
+			(effects
+				(font
+					(size 1.27 1.27)
+				)
+			)
+		)
+		(pin "1"
+		)
+		(instances
+			(project "PCB"
+				(path "/cdb7748a-e4ea-465a-80fd-c707816a3e95"
+					(reference "J3")
+					(unit 1)
+				)

Commit message: commite
Parts:
- C2: footprint (none) -> Capacitor_THT:CP_Radial_D10.0mm_P5.00mm
- J1: footprint Connector_PinHeader_1.00mm:PinHeader_1x06_P1.00mm_Vertical -> Connector_PinHeader_1.00mm:PinHeader_1x05_P1.00mm_Vertical
- J3, J4: footprint (none) -> Taranium-libs:Electromagnet Power Output; symbol Connector:Conn_01x01_Pin -> Connector:Conn_01x02_Pin
Connections:
- net GND: now also J3.2 (Pin_2), J4.2 (Pin_2)
Changed lines of the file:
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@@
 	)
 	(label "OUT1"
-		(at 133.35 81.28 0)
+		(at 132.08 83.82 0)
 		(effects
 			(font
@@
 			)
 		)
-		(property "Footprint" "Connector_PinHeader_1.00mm:PinHeader_1x06_P1.00mm_Vertical"
+		(property "Footprint" "Connector_PinHeader_1.00mm:PinHeader_1x05_P1.00mm_Vertical"
 			(at 31.75 153.67 0)
 			(hide yes)
@@
 	)
 	(symbol
-		(lib_id "Connector:Conn_01x01_Pin")
-		(at 128.27 81.28 0)
+		(lib_id "Connector:Conn_01x02_Pin")
+		(at 127 83.82 0)
 		(unit 1)
 		(body_style 1)
@@
 		(fields_autoplaced yes)
 		(property "Reference" "J4"
-			(at 128.905 76.2 0)
+			(at 127.635 78.74 0)
 			(show_name no)
 			(do_not_autoplace no)
@@
 		)
 		(property "Value" "OUTPUT1"
-			(at 128.905 78.74 0)
-			(show_name no)
-			(do_not_autoplace no)
-			(effects
-				(font
-					(size 1.27 1.27)
-				)
-			)
-		)
-		(property "Footprint" ""
-			(at 128.27 81.28 0)
-			(hide yes)
-			(show_name no)
-			(do_not_autoplace no)
-			(effects
-				(font
-					(size 1.27 1.27)
-				)
-			)
-		)
-		(property "Datasheet" ""
-			(at 128.27 81.28 0)
-			(hide yes)
-			(show_name no)
-			(do_not_autoplace no)
-			(effects
-				(font
-					(size 1.27 1.27)
-				)
-			)
-		)
-		(property "Description" "Generic connector, single row, 01x01, script generated"
-			(at 128.27 81.28 0)
-			(hide yes)
-			(show_name no)
-			(do_not_autoplace no)
-			(effects
-				(font
-					(size 1.27 1.27)
-				)
-			)
-		)
-		(pin "1"
+			(at 127.635 81.28 0)
+			(show_name no)
+			(do_not_autoplace no)
+			(effects
+				(font
+					(size 1.27 1.27)
+				)
+			)
+		)
+		(property "Footprint" "Taranium-libs:Electromagnet Power Output"
+			(at 127 83.82 0)
+			(hide yes)
+			(show_name no)
+			(do_not_autoplace no)
+			(effects
+				(font
+					(size 1.27 1.27)
+				)
+			)
+		)
+		(property "Datasheet" ""
+			(at 127 83.82 0)
+			(hide yes)
+			(show_name no)
+			(do_not_autoplace no)
+			(effects
+				(font
+					(size 1.27 1.27)
+				)
+			)
+		)
+		(property "Description" "Generic connector, single row, 01x02, script generated"
+			(at 127 83.82 0)
+			(hide yes)
+			(show_name no)
+			(do_not_autoplace no)
+			(effects
+				(font
+					(size 1.27 1.27)
+				)
+			)
+		)
+		(pin "1"
+		)
+		(pin "2"
 		)
 		(instances
@@
 			)
 		)
-		(property "Footprint" ""
+		(property "Footprint" "Capacitor_THT:CP_Radial_D10.0mm_P5.00mm"
 			(at 118.11 92.71 0)
 			(hide yes)
@@
 	)
 	(symbol
-		(lib_id "Connector:Conn_01x01_Pin")
+		(lib_id "Connector:Conn_01x02_Pin")
 		(at 127 73.66 0)
 		(unit 1)
@@
 			)
 		)
-		(property "Footprint" ""
+		(property "Footprint" "Taranium-libs:Electromagnet Power Output"
 			(at 127 73.66 0)
 			(hide yes)
@@
 			)
 		)
-		(property "Description" "Generic connector, single row, 01x01, script generated"
+		(property "Description" "Generic connector, single row, 01x02, script generated"
 			(at 127 73.66 0)
 			(hide yes)
@@
 		)
 		(pin "1"
+		)
+		(pin "2"
 		)
 		(instances
@@
 					(unit 1)
 				)
+			)
+		)
+	)
+	(symbol
+		(lib_id "power:GND")
+		(at 132.08 76.2 90)
+		(unit 1)
+		(body_style 1)
+		(exclude_from_sim no)
+		(in_bom yes)
+		(on_board yes)
+		(in_pos_files yes)
+		(dnp no)
+		(fields_autoplaced yes)
+		(property "Reference" "#PWR010"
+			(at 138.43 76.2 0)
+			(hide yes)
+			(show_name no)
+			(do_not_autoplace no)
+			(effects
+				(font
+					(size 1.27 1.27)
+				)
+			)
+		)
+		(property "Value" "GND"
+			(at 135.89 76.1999 90)
+			(show_name no)
+			(do_not_autoplace no)
+			(effects
+				(font
+					(size 1.27 1.27)
+				)
+				(justify right)
+			)
+		)
+		(property "Footprint" ""
+			(at 132.08 76.2 0)
+			(hide yes)
+			(show_name no)
+			(do_not_autoplace no)
+			(effects
+				(font
+					(size 1.27 1.27)
+				)
+			)
+		)
+		(property "Datasheet" ""
+			(at 132.08 76.2 0)
+			(hide yes)
+			(show_name no)
+			(do_not_autoplace no)
+			(effects
+				(font
+					(size 1.27 1.27)
+				)
+			)
+		)
+		(property "Description" "Power symbol creates a global label with name \"GND\" , ground"
+			(at 132.08 76.2 0)
+			(hide yes)
+			(show_name no)
+			(do_not_autoplace no)
+			(effects
+				(font
+					(size 1.27 1.27)
+				)
+			)
+		)
+		(pin "1"
+		)
+		(instances
+			(project "PCB"
+				(path "/cdb7748a-e4ea-465a-80fd-c707816a3e95"
+					(reference "#PWR010")
+					(unit 1)
+				)
+			)
+		)
+	)
+	(symbol
+		(lib_id "power:GND")
+		(at 132.08 86.36 90)
+		(unit 1)
+		(body_style 1)
+		(exclude_from_sim no)
+		(in_bom yes)
+		(on_board yes)
+		(in_pos_files yes)
+		(dnp no)
+		(fields_autoplaced yes)
+		(property "Reference" "#PWR016"
+			(at 138.43 86.36 0)
+			(hide yes)
+			(show_name no)
+			(do_not_autoplace no)
+			(effects
+				(font
+					(size 1.27 1.27)
+				)
+			)
+		)
+		(property "Value" "GND"
+			(at 135.89 86.3599 90)
+			(show_name no)
+			(do_not_autoplace no)
+			(effects
+				(font
+					(size 1.27 1.27)
+				)
+				(justify right)
+			)
+		)
+		(property "Footprint" ""
+			(at 132.08 86.36 0)
+			(hide yes)
+			(show_name no)
+			(do_not_autoplace no)
+			(effects
+				(font
+					(size 1.27 1.27)
+				)
+			)
+		)
+		(property "Datasheet" ""
+			(at 132.08 86.36 0)
+			(hide yes)
+			(show_name no)
+			(do_not_autoplace no)
+			(effects
+				(font
+					(size 1.27 1.27)
+				)
+			)
+		)
+		(property "Description" "Power symbol creates a global label with name \"GND\" , ground"
+			(at 132.08 86.36 0)
+			(hide yes)
+			(show_name no)
+			(do_not_autoplace no)
+			(effects
+				(font
+					(size 1.27 1.27)
+				)
+			)
+		)
+		(pin "1"
+		)
+		(instances
+			(project "PCB"
+				(path "/cdb7748a-e4ea-465a-80fd-c707816a3e95"
+					(reference "#PWR016")
+					(unit 1)
+				)

Commit message: bleh
Parts:
- added C10, C11, C14, C15, C6, C7: 100nf, Capacitor_SMD:C_0402_1005Metric, symbol Device:C_Small
- added C12, C16, C8: 22uf, Capacitor_THT:CP_Radial_D10.0mm_P5.00mm, symbol Device:C_Polarized_Small
- added C13, C5, C9: 22nf, Capacitor_SMD:C_0402_1005Metric, symbol Device:C_Small
- added D2, D3, D4: LED, LED_SMD:LED_0805_2012Metric, symbol Device:LED
- added J10, J6, J8: OUTPUT1, Taranium-libs:Electromagnet Power Output, symbol Connector:Conn_01x02_Pin
- added J5, J7, J9: OUTPUT2, Taranium-libs:Electromagnet Power Output, symbol Connector:Conn_01x02_Pin
- added R10, R13, R7: 2k, Capacitor_SMD:C_0402_1005Metric, symbol Device:R_Small
- added R11, R3, R8: 1k, Capacitor_SMD:C_0402_1005Metric, symbol Device:R_Small
- added R12, R6, R9: 10k, Capacitor_SMD:C_0402_1005Metric, symbol Device:R_Small
- added U3, U5, U7: (no value), Package_TO_SOT_SMD:SOT-353_SC-70-5, symbol Taranium-libs:SN74LVC1G02
- added U4, U6, U8: (no value), Package_SO:HTSSOP-16-1EP_4.4x5mm_P0.65mm_EP3.4x5mm_Mask2.46x2.31mm_ThermalVias, symbol Taranium-libs:DRV8874PWPR
Connections:
- net +24V: now also C10.2, C11.2, C12.1, C14.2, C15.2, C16.1, C6.2, C7.2, C8.1, U4.11 (VM), U6.11 (VM), U8.11 (VM)
- net +3V3: now also R10.1, R12.2, R13.1, R6.2, R7.1, R9.2, U3.5 (VCC), U5.5 (VCC), U7.5 (VCC)
- net GND: now also C11.1, C12.2, C15.1, C16.2, C7.1, C8.2, D2.1 (K), D3.1 (K), D4.1 (K), J10.2 (Pin_2), J5.2 (Pin_2), J6.2 (Pin_2), J7.2 (Pin_2), J8.2 (Pin_2), J9.2 (Pin_2), U3.2 (B), U3.3 (GND), U4.15 (GND), U4.16 (PMODE), U4.6 (IPROPI), U4.7 (IMODE), U4.9 (PGND), U5.2 (B), U5.3 (GND), U6.15 (GND), U6.16 (PMODE), U6.6 (IPROPI), U6.7 (IMODE), U6.9 (PGND), U7.2 (B), U7.3 (GND), U8.15 (GND), U8.16 (PMODE), U8.6 (IPROPI), U8.7 (IMODE), U8.9 (PGND)
- net IO1: now also U3.4 (Y), U4.1 (EN/In1), U5.4 (Y), U6.1 (EN/In1), U7.4 (Y), U8.1 (EN/In1)
- net IO2: now also U4.2 (PH/In2), U6.2 (PH/In2), U8.2 (PH/In2)
- net OUT1: now also J10.1 (Pin_1), J6.1 (Pin_1), J8.1 (Pin_1), U4.8 (OUT1), U6.8 (OUT1), U8.8 (OUT1)
- net OUT2: now also J5.1 (Pin_1), J7.1 (Pin_1), J9.1 (Pin_1), U4.10 (OUT2), U6.10 (OUT2), U8.10 (OUT2)
- net SLEEP: now also R12.1, R6.1, R9.1, U4.3 (nSLEEP), U6.3 (nSLEEP), U8.3 (nSLEEP)
- net IO3: now reaches J1.2 (Pin_2)
- net IO3: now also U3.1 (A)
- net IO4: now reaches J1.3 (Pin_3)
- net IO4: now also U5.1 (A)
- net IO5: now reaches J1.4 (Pin_4)
- net IO5: now also U7.1 (A)
- new net: R10.2, U6.5 (VREF)
- new net: C6.1, U4.12 (VCP)
- new net: C5.2, U4.13 (CPH)
- new net: C5.1, U4.14 (CPL)
- new net: R3.2, U4.4 (nFAULT)
- new net: R7.2, U4.5 (VREF)
- new net: C13.1, U8.14 (CPL)
- new net: C13.2, U8.13 (CPH)
- new net: D3.2 (A), R8.1
- new net: R8.2, U6.4 (nFAULT)
- new net: C10.1, U6.12 (VCP)
- new net: C9.1, U6.14 (CPL)
- new net: C9.2, U6.13 (CPH)
- new net: R13.2, U8.5 (VREF)
- new net: D4.2 (A), R11.1
- new net: C14.1, U8.12 (VCP)
- new net: D2.2 (A), R3.1
- new net: R11.2, U8.4 (nFAULT)
Other:
- moved on the sheet: C1, C2, C3, C4, D1, J1, J2, J3, J4, R2, R4, R5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

Commit message: guh
Parts:
- added H1, H2: MountingHole, MountingHole:MountingHole_2.2mm_M2_Pad_Via, symbol Mechanical:MountingHole
Changed lines of the file:
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@@
+	)
+	(symbol
+		(lib_id "Mechanical:MountingHole")
+		(at 118.11 179.07 0)
+		(unit 1)
+		(body_style 1)
+		(exclude_from_sim no)
+		(in_bom no)
+		(on_board yes)
+		(in_pos_files yes)
+		(dnp no)
+		(fields_autoplaced yes)
+		(property "Reference" "H2"
+			(at 120.65 177.7999 0)
+			(show_name no)
+			(do_not_autoplace no)
+			(effects
+				(font
+					(size 1.27 1.27)
+				)
+				(justify left)
+			)
+		)
+		(property "Value" "MountingHole"
+			(at 120.65 180.3399 0)
+			(show_name no)
+			(do_not_autoplace no)
+			(effects
+				(font
+					(size 1.27 1.27)
+				)
+				(justify left)
+			)
+		)
+		(property "Footprint" "MountingHole:MountingHole_2.2mm_M2_Pad_Via"
+			(at 118.11 179.07 0)
+			(hide yes)
+			(show_name no)
+			(do_not_autoplace no)
+			(effects
+				(font
+					(size 1.27 1.27)
+				)
+			)
+		)
+		(property "Datasheet" ""
+			(at 118.11 179.07 0)
+			(hide yes)
+			(show_name no)
+			(do_not_autoplace no)
+			(effects
+				(font
+					(size 1.27 1.27)
+				)
+			)
+		)
+		(property "Description" "Mounting Hole without connection"
+			(at 118.11 179.07 0)
+			(hide yes)
+			(show_name no)
+			(do_not_autoplace no)
+			(effects
+				(font
+					(size 1.27 1.27)
+				)
+			)
+		)
+		(instances
+			(project "PCB"
+				(path "/cdb7748a-e4ea-465a-80fd-c707816a3e95"
+					(reference "H2")
+					(unit 1)
+				)
+			)
+		)
 	)
 	(symbol
@@
 					(unit 1)
 				)
+			)
+		)
+	)
+	(symbol
+		(lib_id "Mechanical:MountingHole")
+		(at 95.25 179.07 0)
+		(unit 1)
+		(body_style 1)
+		(exclude_from_sim no)
+		(in_bom no)
+		(on_board yes)
+		(in_pos_files yes)
+		(dnp no)
+		(fields_autoplaced yes)
+		(property "Reference" "H1"
+			(at 97.79 177.7999 0)
+			(show_name no)
+			(do_not_autoplace no)
+			(effects
+				(font
+					(size 1.27 1.27)
+				)
+				(justify left)
+			)
+		)
+		(property "Value" "MountingHole"
+			(at 97.79 180.3399 0)
+			(show_name no)
+			(do_not_autoplace no)
+			(effects
+				(font
+					(size 1.27 1.27)
+				)
+				(justify left)
+			)
+		)
+		(property "Footprint" "MountingHole:MountingHole_2.2mm_M2_Pad_Via"
+			(at 95.25 179.07 0)
+			(hide yes)
+			(show_name no)
+			(do_not_autoplace no)
+			(effects
+				(font
+					(size 1.27 1.27)
+				)
+			)
+		)
+		(property "Datasheet" ""
+			(at 95.25 179.07 0)
+			(hide yes)
+			(show_name no)
+			(do_not_autoplace no)
+			(effects
+				(font
+					(size 1.27 1.27)
+				)
+			)
+		)
+		(property "Description" "Mounting Hole without connection"
+			(at 95.25 179.07 0)
+			(hide yes)
+			(show_name no)
+			(do_not_autoplace no)
+			(effects
+				(font
+					(size 1.27 1.27)
+				)
+			)
+		)
+		(instances
+			(project "PCB"
+				(path "/cdb7748a-e4ea-465a-80fd-c707816a3e95"
+					(reference "H1")
+					(unit 1)
+				)

Commit message: commit
Connections:
- net +24V renamed +12V
Changed lines of the file:
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@@
 	)
 	(symbol
-		(lib_id "power:+24V")
+		(lib_id "power:+12V")
 		(at 88.9 38.1 0)
 		(unit 1)
@@
 			)
 		)
-		(property "Value" "+24V"
-			(at 88.9 33.02 0)
+		(property "Value" "+12V"
+			(at 91.44 36.8299 0)
 			(show_name no)
 			(do_not_autoplace no)
@@
 					(size 1.27 1.27)
 				)
+				(justify left)
 			)
 		)
@@
 			)
 		)
-		(property "Description" "Power symbol creates a global label with name \"+24V\""
+		(property "Description" "Power symbol creates a global label with name \"+12V\""
 			(at 88.9 38.1 0)
 			(hide yes)
@@
 	)
 	(symbol
-		(lib_id "power:+24V")
+		(lib_id "power:+12V")
 		(at 242.57 116.84 0)
 		(unit 1)
@@
 			)
 		)
-		(property "Value" "+24V"
-			(at 242.57 111.76 0)
+		(property "Value" "+12V"
+			(at 245.11 115.5699 0)
 			(show_name no)
 			(do_not_autoplace no)
@@
 					(size 1.27 1.27)
 				)
+				(justify left)
 			)
 		)
@@
 			)
 		)
-		(property "Description" "Power symbol creates a global label with name \"+24V\""
+		(property "Description" "Power symbol creates a global label with name \"+12V\""
 			(at 242.57 116.84 0)
 			(hide yes)
@@
 	)
 	(symbol
-		(lib_id "power:+24V")
+		(lib_id "power:+12V")
 		(at 39.37 179.07 0)
 		(unit 1)
@@
 			)
 		)
-		(property "Value" "+24V"
-			(at 39.3699 175.26 90)
+		(property "Value" "+12V"
+			(at 41.91 177.7999 0)
 			(show_name no)
 			(do_not_autoplace no)
@@
 			)
 		)
-		(property "Description" "Power symbol creates a global label with name \"+24V\""
+		(property "Description" "Power symbol creates a global label with name \"+12V\""
 			(at 39.37 179.07 0)
 			(hide yes)
@@
 	)
 	(symbol
-		(lib_id "power:+24V")
+		(lib_id "power:+12V")
 		(at 193.04 39.37 0)
 		(unit 1)
@@
 			)
 		)
-		(property "Value" "+24V"
-			(at 193.04 34.29 0)
+		(property "Value" "+12V"
+			(at 195.58 38.0999 0)
 			(show_name no)
 			(do_not_autoplace no)
@@
 					(size 1.27 1.27)
 				)
+				(justify left)
 			)
 		)
@@
 			)
 		)
-		(property "Description" "Power symbol creates a global label with name \"+24V\""
+		(property "Description" "Power symbol creates a global label with name \"+12V\""
 			(at 193.04 39.37 0)
 			(hide yes)
@@
 	)
 	(symbol
-		(lib_id "power:+24V")
+		(lib_id "power:+12V")
 		(at 91.44 111.76 0)
 		(unit 1)
@@
 			)
 		)
-		(property "Value" "+24V"
-			(at 91.44 106.68 0)
+		(property "Value" "+12V"
+			(at 93.98 110.4899 0)
 			(show_name no)
 			(do_not_autoplace no)
@@
 					(size 1.27 1.27)
 				)
+				(justify left)
 			)
 		)
@@
 			)
 		)
-		(property "Description" "Power symbol creates a global label with name \"+24V\""
+		(property "Description" "Power symbol creates a global label with name \"+12V\""
 			(at 91.44 111.76 0)
 			(hide yes)
