File: PCB-Module/PCB.kicad_pcb (KiCad board)
At the start: 2 copper layers, 68 x 17 mm, 52 parts, among them J1 GPIO/Control, J10 OUTPUT1, J2 POWER, J3 OUTPUT2, J4 OUTPUT1, J5 OUTPUT2, J6 OUTPUT1, J7 OUTPUT2, J8 OUTPUT1, J9 OUTPUT2

Commit message: bleh
Parts:
- moved C13 100.8 mm to (82.4, 27.8)
- moved R11 100.8 mm to (83.4, 37.2)
- moved R12 100.8 mm to (82.4, 37.5)
- moved R8 100.8 mm to (66.4, 37.2)
- moved R9 100.8 mm to (65.4, 37.5)
- moved U1 100.8 mm to (32.5, 32.2)
- moved U4 100.8 mm to (49.5, 32.2)
- moved C12 100.8 mm to (62.5, 26.2)
- moved C2 100.8 mm to (34.3, 25.5)
- moved C5 100.8 mm to (48.4, 27.8)
- moved J1 100.8 mm to (46.5, 40.3)
- moved R5 100.8 mm to (34.0, 37.6)
- moved R7 100.8 mm to (51.0, 37.6)
- moved C1 100.8 mm to (31.6, 27.8)
- moved C11 100.8 mm to (67.8, 26.2)
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Connections:
- C10 pad 2: +24V -> +12V
- C11 pad 2: +24V -> +12V
- C12 pad 1: +24V -> +12V
- C14 pad 2: +24V -> +12V
- C15 pad 2: +24V -> +12V
- C16 pad 1: +24V -> +12V
- C6 pad 2: +24V -> +12V
- C7 pad 2: +24V -> +12V
- C8 pad 1: +24V -> +12V
- U4 pad 11: +24V -> +12V
- U6 pad 11: +24V -> +12V
- U8 pad 11: +24V -> +12V
Routing:
- net +12V: track 11.3 -> 42.1 mm, vias 2 -> 3
- net +24V: track 30.3 -> 0.00 mm
- net GND: track 161.2 -> 166.1 mm, vias 27 -> 28
- net /IO4: track 22.4 -> 20.8 mm
- net /IO5: track 38.7 -> 38.0 mm

Commit message: commit
Parts:
- added J11: Conn_01x01_Pin, Connector_PinHeader_2.54mm:PinHeader_1x01_P2.54mm_Vertical, F.Cu at (90.6, 32.3)
- added Q1: 2SC1623, Package_TO_SOT_SMD:SOT-23, F.Cu at (29.9, 39.4)
- added Q2: 2SC1623, Package_TO_SOT_SMD:SOT-23, F.Cu at (44.9, 35.8)
- added Q3: 2SC1623, Package_TO_SOT_SMD:SOT-23, F.Cu at (61.7, 35.4)
- added Q4: 2SC1623, Package_TO_SOT_SMD:SOT-23, F.Cu at (78.7, 36.0)
- H1, H2: footprint MountingHole:MountingHole_2.2mm_M2_Pad_Via -> MountingHole:MountingHole_2.2mm_M2_Pad_TopOnly
- J1: footprint Connector_PinHeader_1.00mm:PinHeader_1x05_P1.00mm_Vertical -> Connector_PinHeader_2.54mm:PinHeader_1x05_P2.54mm_Vertical
- moved D4 6.75 mm to (87.8, 34.5), turned to -90 degrees
- moved U5 4.20 mm to (61.8, 31.9), turned to 90 degrees
- moved U3 3.58 mm to (45.2, 32.5), turned to 90 degrees
- moved U7 3.42 mm to (78.8, 32.7), turned to 90 degrees
- moved H2 3.22 mm to (39.7, 32.1)
- moved J2 1.54 mm to (27.7, 29.8)
- moved R4 0.61 mm to (31.9, 37.1)
- moved R2 0.48 mm to (32.9, 37.2)
- moved D2 0.39 mm to (53.6, 37.3)
- moved U2 0.35 mm to (28.1, 35.8)
- moved R5 0.31 mm to (34.4, 37.6)
Connections:
- C10 pad 1: Net-(U1-VCP) -> Net-(U6-VCP)
- C13 pad 1: Net-(U1-CPL) -> Net-(U8-CPL)
- C13 pad 2: Net-(U1-CPH) -> Net-(U8-CPH)
- C14 pad 1: Net-(U1-VCP) -> Net-(U8-VCP)
- C5 pad 1: Net-(U1-CPL) -> Net-(U4-CPL)
- C5 pad 2: Net-(U1-CPH) -> Net-(U4-CPH)
- C6 pad 1: Net-(U1-VCP) -> Net-(U4-VCP)
- C9 pad 1: Net-(U1-CPL) -> Net-(U6-CPL)
- C9 pad 2: Net-(U1-CPH) -> Net-(U6-CPH)
- D2 pad 2: Net-(D1-A) -> Net-(D2-A)
- D3 pad 2: Net-(D1-A) -> Net-(D3-A)
- D4 pad 2: Net-(D1-A) -> Net-(D4-A)
- R10 pad 2: Net-(U1-VREF) -> Net-(U6-VREF)
- R11 pad 1: Net-(D1-A) -> Net-(D4-A)
- R11 pad 2: Net-(U1-nFAULT) -> Net-(U8-nFAULT)
- R13 pad 2: Net-(U1-VREF) -> Net-(U8-VREF)
- R3 pad 1: Net-(D1-A) -> Net-(D2-A)
- R3 pad 2: Net-(U1-nFAULT) -> Net-(U4-nFAULT)
- R7 pad 2: Net-(U1-VREF) -> Net-(U4-VREF)
- R8 pad 1: Net-(D1-A) -> Net-(D3-A)
- R8 pad 2: Net-(U1-nFAULT) -> Net-(U6-nFAULT)
- U1 pad 1: /IO1 -> /OUT1
- U1 pad 2: /IO2 -> /TOUT1
- U2 pad 1: /IO2 -> /TOUT1
- U2 pad 4: /IO1 -> /OUT1
- U3 pad 1: /IO3 -> /TOUT2
- U3 pad 4: /IO1 -> /OUT2
- U4 pad 1: /IO1 -> /OUT2
- U4 pad 12: Net-(U1-VCP) -> Net-(U4-VCP)
- U4 pad 13: Net-(U1-CPH) -> Net-(U4-CPH)
- U4 pad 14: Net-(U1-CPL) -> Net-(U4-CPL)
- U4 pad 2: /IO3 -> /TOUT2
- U4 pad 4: Net-(U1-nFAULT) -> Net-(U4-nFAULT)
- U4 pad 5: Net-(U1-VREF) -> Net-(U4-VREF)
- U5 pad 1: /IO4 -> /TOUT3
- U5 pad 4: /IO1 -> /OUT3
- U6 pad 1: /IO1 -> /OUT3
- U6 pad 12: Net-(U1-VCP) -> Net-(U6-VCP)
- U6 pad 13: Net-(U1-CPH) -> Net-(U6-CPH)
- U6 pad 14: Net-(U1-CPL) -> Net-(U6-CPL)
- U6 pad 2: /IO4 -> /TOUT3
- U6 pad 4: Net-(U1-nFAULT) -> Net-(U6-nFAULT)
- U6 pad 5: Net-(U1-VREF) -> Net-(U6-VREF)
- U7 pad 1: /IO5 -> /TOUT4
- U7 pad 4: /IO1 -> /OUT4
- U8 pad 1: /IO1 -> /OUT4
- U8 pad 12: Net-(U1-VCP) -> Net-(U8-VCP)
- U8 pad 13: Net-(U1-CPH) -> Net-(U8-CPH)
- U8 pad 14: Net-(U1-CPL) -> Net-(U8-CPL)
- U8 pad 2: /IO5 -> /TOUT4
- U8 pad 4: Net-(U1-nFAULT) -> Net-(U8-nFAULT)
- U8 pad 5: Net-(U1-VREF) -> Net-(U8-VREF)
Routing:
- net /ROW: track 0.00 -> 69.6 mm, vias 0 -> 5
- net /IO1: track 17.2 -> 0.00 mm
- net Net-(D1-A): track 19.5 -> 4.90 mm, vias 8 -> 2
- net Net-(U1-VCP): track 15.1 -> 3.71 mm
- net +3V3: track 91.5 -> 101.8 mm, vias 8 -> 10
- net GND: track 166.1 -> 157.0 mm, vias 28 -> 25
- net Net-(U1-VREF): track 10.2 -> 2.84 mm
- net /IO4: track 20.8 -> 14.1 mm
- net /TOUT3: track 0.00 -> 6.62 mm
- net /IO5: track 38.0 -> 31.4 mm
- net /TOUT4: track 0.00 -> 5.98 mm
- net /TOUT2: track 0.00 -> 5.62 mm
- net Net-(D4-A): track 0.00 -> 5.56 mm, vias 0 -> 2
- net Net-(U1-CPL): track 7.26 -> 1.78 mm
- net /IO2: track 22.7 -> 17.4 mm
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