File: PCB-Module/PCB.kicad_sch (KiCad schematic)
At the start: 52 parts, among them J1 GPIO/Control, J10 OUTPUT1, J2 POWER, J3 OUTPUT2, J4 OUTPUT1, J5 OUTPUT2, J6 OUTPUT1, J7 OUTPUT2, J8 OUTPUT1, J9 OUTPUT2

Commit message: commit
Parts:
- added J11: Conn_01x01_Pin, Connector_PinHeader_2.54mm:PinHeader_1x01_P2.54mm_Vertical, symbol Connector:Conn_01x01_Pin
- added Q1, Q2, Q3, Q4: 2SC1623, Package_TO_SOT_SMD:SOT-23, symbol Transistor_BJT:BC817
- C12, C16, C2, C8: footprint Capacitor_THT:CP_Radial_D10.0mm_P5.00mm -> Capacitor_THT:CP_Radial_D5.0mm_P2.00mm
- H1, H2: footprint MountingHole:MountingHole_2.2mm_M2_Pad_Via -> MountingHole:MountingHole_2.2mm_M2_Pad_TopOnly
- J1: footprint Connector_PinHeader_1.00mm:PinHeader_1x05_P1.00mm_Vertical -> Connector_PinHeader_2.54mm:PinHeader_1x05_P2.54mm_Vertical
Connections:
- net IO2: now also Q1.1 (B); no longer U1.2 (PH/In2), U2.1 (A), U4.2 (PH/In2), U6.2 (PH/In2), U8.2 (PH/In2)
- net IO3: now also Q2.1 (B); no longer U3.1 (A)
- net IO4: now also Q3.1 (B); no longer U5.1 (A)
- net IO5: now also Q4.1 (B); no longer U7.1 (A)
- net OUT1: now also U1.1 (EN/In1), U2.4 (Y)
- net OUT2: now also U3.4 (Y), U4.1 (EN/In1)
- removed net IO1: U1.1 (EN/In1), U2.4 (Y), U3.4 (Y), U4.1 (EN/In1), U5.4 (Y), U6.1 (EN/In1), U7.4 (Y), U8.1 (EN/In1)
- new net OUT3: U5.4 (Y), U6.1 (EN/In1)
- new net OUT4: U7.4 (Y), U8.1 (EN/In1)
- new net ROW: J11.1 (Pin_1), Q1.3 (C), Q2.3 (C), Q3.3 (C), Q4.3 (C)
- new net TOUT1: Q1.2 (E), U1.2 (PH/In2), U2.1 (A)
- new net TOUT2: Q2.2 (E), U3.1 (A), U4.2 (PH/In2)
- new net TOUT3: Q3.2 (E), U5.1 (A), U6.2 (PH/In2)
- new net TOUT4: Q4.2 (E), U7.1 (A), U8.2 (PH/In2)
