File: PCB-PD/PCB-PD.kicad_pcb (KiCad board)
At the start: 2 copper layers, 106 parts, among them SW1 SW_Push, U1 SCT2650STE, U10 MCP23017, U11 MCP23017, U12 MCP23017, U13 MCP23017, U14 MCP23017, U15 MCP23017, U16 MCP23017, U17 MCP23017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

Commit message: end me
Parts:
- added D3: C48192, Taranium-libs:USB-C-SMD_20P-P0.50-L6.5-W8.9, F.Cu at (89.5, 68.9)
- moved C25 32.6 mm to (64.2, 97.5)
- moved C26 32.6 mm to (64.2, 99.4)
- moved C27 32.6 mm to (64.2, 101.4)
- moved C28 32.6 mm to (64.2, 103.4)
- moved C3 32.6 mm to (57.8, 97.5)
- moved C31 32.6 mm to (64.2, 105.4)
- moved C32 32.6 mm to (64.2, 107.3)
- moved C34 32.6 mm to (67.5, 97.5)
- moved C35 32.6 mm to (67.5, 99.4)
- moved C36 32.6 mm to (67.5, 101.4)
- moved C37 32.6 mm to (67.5, 103.4)
- moved C38 32.6 mm to (67.5, 105.4)
- moved C39 32.6 mm to (67.5, 107.3)
- moved C5 32.6 mm to (57.8, 99.4)
- moved C6 32.6 mm to (57.8, 101.4)
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Connections:
- U2 pad 6: unconnected-(U2-GPIO4-Pad6) -> /SLEEP

Commit message: commit
Parts:
- removed C34, C35, C36, C37, C38, C39, C40, C41, C42, C43, C44, C45, C46, C47: 100nf, Capacitor_SMD:C_0402_1005Metric_Pad0.74x0.62mm_HandSolder
- removed R18, R21, R22, R24, R25, R26, R27, R28, R29, R30, R31, R32, R33, R34, R35, R36, R37, R38, R39, R40, R41, R42, R43: 2.2k, Resistor_SMD:R_0402_1005Metric_Pad0.72x0.64mm_HandSolder
- removed U10, U11, U12, U13, U14, U15, U16, U17, U18, U19, U20, U21, U8, U9: MCP23017, Package_DFN_QFN:QFN-28-1EP_6x6mm_P0.65mm_EP4.25x4.25mm
- added H1: MountingHole, MountingHole:MountingHole_3.2mm_M3_Pad_Via, F.Cu at (128.1, 114.7)
- added H2: MountingHole, MountingHole:MountingHole_3.2mm_M3_Pad_Via, F.Cu at (128.1, 122.6)
- added H3: MountingHole, MountingHole:MountingHole_3.2mm_M3_Pad_Via, F.Cu at (128.1, 130.6)
- added H4: MountingHole, MountingHole:MountingHole_3.2mm_M3_Pad_Via, F.Cu at (128.1, 138.5)
- added J1: Conn_Receptacle_3P_Protected, Taranium-libs:240V Power Outlet, F.Cu at (100.0, 46.4)
- added J10: Conn_01x20_Pin, Connector_PinHeader_2.54mm:PinHeader_1x20_P2.54mm_Vertical, F.Cu at (200.0, 79.7)
- added J11: Conn_01x12_Pin, Connector_PinHeader_2.54mm:PinHeader_1x12_P2.54mm_Vertical, F.Cu at (134.4, 113.0)
- added J2: USB_C_Receptacle_USB2.0_14P, Taranium-libs:USB-C-SMD_20P-P0.50-L6.5-W8.9, F.Cu at (112.9, 73.8)
- added J6: +12V, Taranium-libs:5P_Screw_Terminal, F.Cu at (184.3, 85.4)
- added J7: +3V3, Taranium-libs:5P_Screw_Terminal, F.Cu at (184.3, 93.3)
- added J8: GND, Taranium-libs:5P_Screw_Terminal, F.Cu at (184.3, 101.2)
- added J9: Conn_01x20_Pin, Connector_PinHeader_2.54mm:PinHeader_1x20_P2.54mm_Vertical, F.Cu at (95.0, 82.7)
- added R12: 10k, Resistor_SMD:R_01005_0402Metric, F.Cu at (190.1, 46.5)
- added R15: 300, Resistor_SMD:R_01005_0402Metric, F.Cu at (190.1, 48.1)
- added R16: 10k, Resistor_SMD:R_01005_0402Metric, F.Cu at (190.1, 49.8)
- added SW2: SW_Push, Taranium-libs:C720477, F.Cu at (179.6, 64.4)
- added SW3: SW_Push, Taranium-libs:C720477, F.Cu at (160.5, 71.5)
- C11, C12, C13, C14, C15, C16, C17, C29, C30, C4: footprint Capacitor_SMD:C_0201_0603Metric_Pad0.64x0.40mm_HandSolder -> Capacitor_SMD:C_0603_1608Metric_Pad1.08x0.95mm_HandSolder
- D1: footprint Diode_THT:Diode_Bridge_Round_D9.8mm -> Taranium-libs:DIO-BG-TH_KBPC25
- R10, R9: value 22 -> 27
- R17: value 2.2k -> 300; footprint Resistor_SMD:R_0402_1005Metric_Pad0.72x0.64mm_HandSolder -> Resistor_SMD:R_01005_0402Metric
- moved R17 155.8 mm to (190.1, 51.4)
- moved R6 150.2 mm to (187.2, 71.1)
- moved R11 144.9 mm to (185.8, 134.4)
- moved R13 144.9 mm to (185.8, 136.4)
- moved R14 144.9 mm to (185.8, 138.4)
- moved R10 144.4 mm to (182.6, 142.4)
- moved R9 144.4 mm to (182.6, 140.4)
- moved R7 143.7 mm to (182.6, 136.4)
- moved R8 143.7 mm to (182.6, 138.4)
- moved R4 138.4 mm to (172.7, 59.5), turned to -90 degrees
- moved R5 134.4 mm to (162.7, 47.7)
- moved R3 128.5 mm to (163.4, 61.1), turned to -90 degrees
- moved R1 126.9 mm to (161.8, 57.2), turned to -90 degrees
- moved R2 125.6 mm to (160.6, 59.5), turned to -90 degrees
- moved C3 122.1 mm to (173.8, 59.5), turned to -90 degrees
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Connections:
- R17 pad 1: +3V3 -> Net-(R16-Pad2)
- R17 pad 2: Net-(U7-A0) -> Net-(U7-~{RESET})
- U2 pad 4: /SDA1 -> /SLEEP
- U2 pad 5: /SCL1 -> unconnected-(U2-GPIO3-Pad5)
- U2 pad 6: /SLEEP -> unconnected-(U2-GPIO4-Pad6)
- U6 pad 14: unconnected-(U6-~{RESET}-Pad14) -> Net-(U6-~{RESET})
- U6 pad 29: unconnected-(U6-EP-Pad29) -> GND
- U7 pad 11: Net-(U7-A0) -> +3V3
- U7 pad 12: GND -> +3V3
- U7 pad 13: GND -> +3V3
- U7 pad 14: unconnected-(U7-~{RESET}-Pad14) -> Net-(U7-~{RESET})
- U7 pad 29: unconnected-(U7-EP-Pad29) -> GND
Routing:
- net +12V: track 0.00 -> 9.16 mm
