File: PCB-PD/PCB-PD.kicad_sch (KiCad schematic)
At the start: 28 parts, among them J1 Conn_Receptacle_3P_Protected, T1 Transformer_1P_1S, U1 SCT2650STE, Y1 Crystal_GND24_Small

Commit message: bleh
Parts:
- removed Y1: Crystal_GND24_Small, symbol Device:Crystal_GND24_Small
- added C16, C17: 10uf, Capacitor_SMD:C_0201_0603Metric_Pad0.64x0.40mm_HandSolder, symbol Device:C_Small
- added C18, C20, C21, C23, C24, C25, C26, C27, C28, C31, C32, C33, C34, C35, C36, C37, C38, C39, C40, C41, C42, C43, C44, C45, C46, C47: 100nf, Capacitor_SMD:C_0402_1005Metric_Pad0.74x0.62mm_HandSolder, symbol Device:C_Small
- added C19, C22: 1uf, Capacitor_SMD:C_0402_1005Metric_Pad0.74x0.62mm_HandSolder, symbol Device:C_Small
- added C29, C30: 15pf, Capacitor_SMD:C_0201_0603Metric_Pad0.64x0.40mm_HandSolder, symbol Device:C_Small
- added D3: C48192, symbol Device:D_Small
- added J2: USB_C_Receptacle_USB2.0_14P, symbol Connector:USB_C_Receptacle_USB2.0_14P
- added R10, R9: 22, Resistor_SMD:R_0402_1005Metric_Pad0.72x0.64mm_HandSolder, symbol Device:R_Small
- added R11: 1k, Resistor_SMD:R_0402_1005Metric_Pad0.72x0.64mm_HandSolder, symbol Device:R_Small
- added R13: 10k, Resistor_SMD:R_0402_1005Metric_Pad0.72x0.64mm_HandSolder, symbol Device:R_Small
- added R14: 300, Resistor_SMD:R_0402_1005Metric_Pad0.72x0.64mm_HandSolder, symbol Device:R_Small
- added R17, R18, R21, R22, R24, R25, R26, R27, R28, R29, R30, R31, R32, R33, R34, R35, R36, R37, R38, R39, R40, R41, R42, R43: 2.2k, Resistor_SMD:R_0402_1005Metric_Pad0.72x0.64mm_HandSolder, symbol Device:R_Small
- added R7, R8: 5.1k, Resistor_SMD:R_0402_1005Metric_Pad0.72x0.64mm_HandSolder, symbol Device:R_Small
- added SW1: SW_Push, Taranium-libs:C720477, symbol Switch:SW_Push
- added U10, U11, U12, U13, U14, U15, U16, U17, U18, U19, U20, U21, U6, U7, U8, U9: MCP23017, Package_DFN_QFN:QFN-28-1EP_6x6mm_P0.65mm_EP4.25x4.25mm, symbol Interface_Expansion:MCP23017x-x-ML
- added U2: RP2040, Package_DFN_QFN:QFN-56-1EP_7x7mm_P0.4mm_EP3.2x3.2mm, symbol MCU_RaspberryPi:RP2040
- added U3: MCP1700, Package_TO_SOT_SMD:SOT-23, symbol Regulator_Linear:MCP1700x-120xxTT
- added U4: USBLC6-2SC6, Package_TO_SOT_SMD:SOT-23-6, symbol Power_Protection:USBLC6-2SC6
- added U5: W25Q16JVSS, Package_SO:SOIC-8_5.3x5.3mm_P1.27mm, symbol Memory_Flash:W25Q16JVSS
- added Y1: 12mHz, Taranium-libs:CRYSTAL-SMD_4P-L3.2-W2.5-BL, symbol Device:Crystal_GND24
- C10, C3, C5, C6, C7, C8, C9: footprint (none) -> Capacitor_SMD:C_0402_1005Metric_Pad0.74x0.62mm_HandSolder
- C11, C12, C13, C14, C15, C4: footprint (none) -> Capacitor_SMD:C_0201_0603Metric_Pad0.64x0.40mm_HandSolder
- R1, R2, R3, R4, R5, R6: footprint (none) -> Resistor_SMD:R_0402_1005Metric_Pad0.72x0.64mm_HandSolder
Connections:
- net +3V3: now also C17.1, C22.2, C23.2, C24.2, C25.2, C26.2, C27.2, C28.2, C31.2, C32.2, C33.2, C34.2, C35.2, C36.2, C37.2, C38.2, C39.2, C40.2, C41.2, C42.2, C43.2, C44.2, C45.2, C46.2, C47.2, R13.2, R17.1, R18.1, R21.1, R22.1, R24.1, R25.1, R26.1, R27.1, R28.1, R29.1, R30.1, R31.1, R32.1, R33.1, R34.1, R35.1, R36.1, R37.1, R38.1, R39.1, R40.1, R41.1, R42.1, R43.1, U10.5 (V_{DD}), U11.5 (V_{DD}), U12.5 (V_{DD}), U13.5 (V_{DD}), U14.5 (V_{DD}), U15.5 (V_{DD}), U16.5 (V_{DD}), U17.5 (V_{DD}), U18.5 (V_{DD}), U19.5 (V_{DD}), U2.1 (IOVDD), U2.10 (IOVDD), U2.22 (IOVDD), U2.23 (DVDD), U2.33 (IOVDD), U2.42 (IOVDD), U2.44 (VREG_VIN), U2.45 (VREG_VOUT), U2.49 (IOVDD), U2.50 (DVDD), U20.5 (V_{DD}), U21.5 (V_{DD}), U3.2 (VO), U5.8 (VCC), U6.5 (V_{DD}), U7.5 (V_{DD}), U8.5 (V_{DD}), U9.5 (V_{DD})
- net GND: now also C16.2, C17.2, C18.2, C19.1, C20.1, C21.1, C22.1, C23.1, C24.1, C25.1, C26.1, C27.1, C28.1, C29.2, C30.2, C31.1, C32.1, C33.1, C34.1, C35.1, C36.1, C37.1, C38.1, C39.1, C40.1, C41.1, C42.1, C43.1, C44.1, C45.1, C46.1, C47.1, J2.A1 (GND), J2.A12 (GND), J2.B1 (GND), J2.B12 (GND), J2.SH (SHIELD), R7.2, R8.2, SW1.1, U10.11 (A0), U10.12 (A1), U10.6 (V_{SS}), U11.12 (A1), U11.6 (V_{SS}), U12.11 (A0), U12.6 (V_{SS}), U13.6 (V_{SS}), U14.11 (A0), U14.12 (A1), U14.6 (V_{SS}), U15.12 (A1), U15.6 (V_{SS}), U16.11 (A0), U16.6 (V_{SS}), U17.6 (V_{SS}), U18.11 (A0), U18.12 (A1), U18.13 (A2), U18.6 (V_{SS}), U19.12 (A1), U19.13 (A2), U19.6 (V_{SS}), U2.57 (GND), U20.11 (A0), U20.13 (A2), U20.6 (V_{SS}), U21.13 (A2), U21.6 (V_{SS}), U3.1 (GND), U4.2 (GND), U5.4 (GND), U6.11 (A0), U6.12 (A1), U6.13 (A2), U6.6 (V_{SS}), U7.12 (A1), U7.13 (A2), U7.6 (V_{SS}), U8.11 (A0), U8.13 (A2), U8.6 (V_{SS}), U9.13 (A2), U9.6 (V_{SS}), Y1.2 (G), Y1.4 (G)
- new net: R24.2, U9.12 (A1)
- new net: R26.2, U21.11 (A0)
- new net: R41.2, U17.11 (A0)
- new net: C16.1, D3.2 (A), J2.A4 (VBUS), J2.A9 (VBUS), J2.B4 (VBUS), J2.B9 (VBUS), U3.3 (VI)
- new net: J2.A5 (CC1), R7.1
- new net: J2.A6 (D+), J2.B6 (D+), U4.3 (I/O2)
- new net: J2.A7 (D-), J2.B7 (D-), U4.1 (I/O1)
- new net: J2.B5 (CC2), R8.1
- new net: R27.2, U21.12 (A1)
- new net: R28.2, U10.13 (A2)
- new net: C30.1, R11.1, Y1.3
- new net: R39.2, U16.12 (A1)
- new net: R18.2, U19.11 (A0)
- new net: R30.2, U14.13 (A2)
- new net: R40.2, U16.13 (A2)
- new net: R33.2, U12.12 (A1)
- new net: R36.2, U13.12 (A1)
- new net: R29.2, U11.11 (A0)
- new net: R22.2, U20.12 (A1)
- new net: R14.1, U2.26 (RUN)
- new net: R34.2, U12.13 (A2)
- new net: R21.2, U8.12 (A1)
- new net: R9.2, U2.46 (USB_DM)
- new net: R10.2, U2.47 (USB_DP)
- new net: R38.2, U15.13 (A2)
- new net: R32.2, U15.11 (A0)
- new net: R25.2, U9.11 (A0)
- new net: R17.2, U7.11 (A0)
- new net: R35.2, U13.11 (A0)
- new net: R37.2, U13.13 (A2)
- new net: R42.2, U17.12 (A1)
- new net: R43.2, U17.13 (A2)
- new net: R31.2, U11.13 (A2)
- new net +1V1: C19.2, C20.2, C21.2, U2.43 (ADC_AVDD), U2.48 (USB_VDD)
- new net +5V: C18.1, D3.1 (K), U4.5 (VBUS)
- new net 00A0: U18.17 (GPA0), U6.17 (GPA0)
- new net 00A1: U18.18 (GPA1), U6.18 (GPA1)
- new net 00A2: U18.19 (GPA2), U6.19 (GPA2)
- new net 00A3: U18.20 (GPA3), U6.20 (GPA3)
- new net 00A4: U18.21 (GPA4), U6.21 (GPA4)
- new net 00A5: U18.22 (GPA5), U6.22 (GPA5)
- new net 00A6: U18.23 (GPA6), U6.23 (GPA6)
- new net 00A7: U18.24 (GPA7), U6.24 (GPA7)
- new net 00B0: U18.25 (GPB0), U6.25 (GPB0)
- new net 00B1: U18.26 (GPB1), U6.26 (GPB1)
- new net 00B2: U18.27 (GPB2), U6.27 (GPB2)
- new net 00B3: U18.28 (GPB3), U6.28 (GPB3)
- new net 00B4: U18.1 (GPB4), U6.1 (GPB4)
- new net 00B5: U18.2 (GPB5), U6.2 (GPB5)
- new net 00B6: U18.3 (GPB6), U6.3 (GPB6)
- new net 00B7: U18.4 (GPB7), U6.4 (GPB7)
- new net 01A0: U19.17 (GPA0), U7.17 (GPA0)
- new net 01A1: U19.18 (GPA1), U7.18 (GPA1)
- new net 01A2: U19.19 (GPA2), U7.19 (GPA2)
- new net 01A3: U19.20 (GPA3), U7.20 (GPA3)
- new net 01A4: U19.21 (GPA4), U7.21 (GPA4)
- new net 01A5: U19.22 (GPA5), U7.22 (GPA5)
- new net 01A6: U19.23 (GPA6), U7.23 (GPA6)
- new net 01A7: U19.24 (GPA7), U7.24 (GPA7)
- new net 01B0: U19.25 (GPB0), U7.25 (GPB0)
- new net 01B1: U19.26 (GPB1), U7.26 (GPB1)
- new net 01B2: U19.27 (GPB2), U7.27 (GPB2)
- new net 01B3: U19.28 (GPB3), U7.28 (GPB3)
- new net 01B4: U19.1 (GPB4), U7.1 (GPB4)
- new net 01B5: U19.2 (GPB5), U7.2 (GPB5)
- new net 01B6: U19.3 (GPB6), U7.3 (GPB6)
- new net 01B7: U19.4 (GPB7), U7.4 (GPB7)
- new net 02A0: U20.17 (GPA0), U8.17 (GPA0)
- new net 02A1: U20.18 (GPA1), U8.18 (GPA1)
- new net 02A2: U20.19 (GPA2), U8.19 (GPA2)
- new net 02A3: U20.20 (GPA3), U8.20 (GPA3)
- new net 02A4: U20.21 (GPA4), U8.21 (GPA4)
- new net 02A5: U20.22 (GPA5), U8.22 (GPA5)
- new net 02A6: U20.23 (GPA6), U8.23 (GPA6)
- new net 02A7: U20.24 (GPA7), U8.24 (GPA7)
- new net 02B0: U20.25 (GPB0), U8.25 (GPB0)
- new net 02B1: U20.26 (GPB1), U8.26 (GPB1)
- new net 02B2: U20.27 (GPB2), U8.27 (GPB2)
- new net 02B3: U20.28 (GPB3), U8.28 (GPB3)
- new net 02B4: U20.1 (GPB4), U8.1 (GPB4)
- new net 02B5: U20.2 (GPB5), U8.2 (GPB5)
- new net 02B6: U20.3 (GPB6), U8.3 (GPB6)
- new net 02B7: U20.4 (GPB7), U8.4 (GPB7)
- new net 03A0: U21.17 (GPA0), U9.17 (GPA0)
- new net 03A1: U21.18 (GPA1), U9.18 (GPA1)
- new net 03A2: U21.19 (GPA2), U9.19 (GPA2)
- new net 03A3: U21.20 (GPA3), U9.20 (GPA3)
- new net 03A4: U21.21 (GPA4), U9.21 (GPA4)
- new net 03A5: U21.22 (GPA5), U9.22 (GPA5)
- new net 03A6: U21.23 (GPA6), U9.23 (GPA6)
- new net 03A7: U21.24 (GPA7), U9.24 (GPA7)
- new net 03B0: U21.25 (GPB0), U9.25 (GPB0)
- new net 03B1: U21.26 (GPB1), U9.26 (GPB1)
- new net 03B2: U21.27 (GPB2), U9.27 (GPB2)
- new net 03B3: U21.28 (GPB3), U9.28 (GPB3)
- new net 03B4: U21.1 (GPB4), U9.1 (GPB4)
- new net 03B5: U21.2 (GPB5), U9.2 (GPB5)
- new net 03B6: U21.3 (GPB6), U9.3 (GPB6)
- new net 03B7: U21.4 (GPB7), U9.4 (GPB7)
- new net 04A0: U10.17 (GPA0), U14.17 (GPA0)
- new net 04A1: U10.18 (GPA1), U14.18 (GPA1)
- new net 04A2: U10.19 (GPA2), U14.19 (GPA2)
- new net 04A3: U10.20 (GPA3), U14.20 (GPA3)
- new net 04A4: U10.21 (GPA4), U14.21 (GPA4)
- new net 04A5: U10.22 (GPA5), U14.22 (GPA5)
- new net 04A6: U10.23 (GPA6), U14.23 (GPA6)
- new net 04A7: U10.24 (GPA7), U14.24 (GPA7)
- new net 04B0: U10.25 (GPB0), U14.25 (GPB0)
- new net 04B1: U10.26 (GPB1), U14.26 (GPB1)
- new net 04B2: U10.27 (GPB2), U14.27 (GPB2)
- new net 04B3: U10.28 (GPB3), U14.28 (GPB3)
- new net 04B4: U10.1 (GPB4), U14.1 (GPB4)
- new net 04B5: U10.2 (GPB5), U14.2 (GPB5)
- new net 04B6: U10.3 (GPB6), U14.3 (GPB6)
- new net 04B7: U10.4 (GPB7), U14.4 (GPB7)
- new net 05A0: U11.17 (GPA0), U15.17 (GPA0)
- new net 05A1: U11.18 (GPA1), U15.18 (GPA1)
- new net 05A2: U11.19 (GPA2), U15.19 (GPA2)
- new net 05A3: U11.20 (GPA3), U15.20 (GPA3)
- new net 05A4: U11.21 (GPA4), U15.21 (GPA4)
- new net 05A5: U11.22 (GPA5), U15.22 (GPA5)
- new net 05A6: U11.23 (GPA6), U15.23 (GPA6)
- new net 05A7: U11.24 (GPA7), U15.24 (GPA7)
- new net 05B0: U11.25 (GPB0), U15.25 (GPB0)
- new net 05B1: U11.26 (GPB1), U15.26 (GPB1)
- new net 05B2: U11.27 (GPB2), U15.27 (GPB2)
- new net 05B3: U11.28 (GPB3), U15.28 (GPB3)
- new net 05B4: U11.1 (GPB4), U15.1 (GPB4)
- new net 05B5: U11.2 (GPB5), U15.2 (GPB5)
- new net 05B6: U11.3 (GPB6), U15.3 (GPB6)
- new net 05B7: U11.4 (GPB7), U15.4 (GPB7)
- new net 06A0: U12.17 (GPA0), U16.17 (GPA0)
- new net 06A1: U12.18 (GPA1), U16.18 (GPA1)
- new net 06A2: U12.19 (GPA2), U16.19 (GPA2)
- new net 06A3: U12.20 (GPA3), U16.20 (GPA3)
- new net 06A4: U12.21 (GPA4), U16.21 (GPA4)
- new net 06A5: U12.22 (GPA5), U16.22 (GPA5)
- new net 06A6: U12.23 (GPA6), U16.23 (GPA6)
- new net 06A7: U12.24 (GPA7), U16.24 (GPA7)
- new net 06B0: U12.25 (GPB0), U16.25 (GPB0)
- new net 06B1: U12.26 (GPB1), U16.26 (GPB1)
- new net 06B2: U12.27 (GPB2), U16.27 (GPB2)
- new net 06B3: U12.28 (GPB3), U16.28 (GPB3)
- new net 06B4: U12.1 (GPB4), U16.1 (GPB4)
- new net 06B5: U12.2 (GPB5), U16.2 (GPB5)
- new net 06B6: U12.3 (GPB6), U16.3 (GPB6)
- new net 06B7: U12.4 (GPB7), U16.4 (GPB7)
- new net 07A0: U13.17 (GPA0), U17.17 (GPA0)
- new net 07A1: U13.18 (GPA1), U17.18 (GPA1)
- new net 07A2: U13.19 (GPA2), U17.19 (GPA2)
- new net 07A3: U13.20 (GPA3), U17.20 (GPA3)
- new net 07A4: U13.21 (GPA4), U17.21 (GPA4)
- new net 07A5: U13.22 (GPA5), U17.22 (GPA5)
- new net 07A6: U13.23 (GPA6), U17.23 (GPA6)
- new net 07A7: U13.24 (GPA7), U17.24 (GPA7)
- new net 07B0: U13.25 (GPB0), U17.25 (GPB0)
- new net 07B1: U13.26 (GPB1), U17.26 (GPB1)
- new net 07B2: U13.27 (GPB2), U17.27 (GPB2)
- new net 07B3: U13.28 (GPB3), U17.28 (GPB3)
- new net 07B4: U13.1 (GPB4), U17.1 (GPB4)
- new net 07B5: U13.2 (GPB5), U17.2 (GPB5)
- new net 07B6: U13.3 (GPB6), U17.3 (GPB6)
- new net 07B7: U13.4 (GPB7), U17.4 (GPB7)
- new net CLK: U2.52 (QSPI_SCLK), U5.6 (CLK)
- new net DN: R9.1, U4.6 (I/O1)
- new net DP: R10.1, U4.4 (I/O2)
- new net RUN: R13.1, R14.2, SW1.2
- new net SCL0: U10.9 (SDA), U11.9 (SDA), U12.9 (SDA), U13.9 (SDA), U2.3 (GPIO1), U6.9 (SDA), U7.9 (SDA), U8.9 (SDA), U9.9 (SDA)
- new net SCL1: U14.9 (SDA), U15.9 (SDA), U16.9 (SDA), U17.9 (SDA), U18.9 (SDA), U19.9 (SDA), U2.5 (GPIO3), U20.9 (SDA), U21.9 (SDA)
- new net SD0: U2.53 (QSPI_SD0), U5.5 (DI/IO_{0})
- new net SD1: U2.55 (QSPI_SD1), U5.2 (DO/IO_{1})
- new net SD2: U2.54 (QSPI_SD2), U5.3 (~{WP}/IO_{2})
- new net SD3: U2.51 (QSPI_SD3), U5.7 (~{HOLD}/~{RESET}/IO_{3})
- new net SDA0: U10.8 (SCK), U11.8 (SCK), U12.8 (SCK), U13.8 (SCK), U2.2 (GPIO0), U6.8 (SCK), U7.8 (SCK), U8.8 (SCK), U9.8 (SCK)
- new net SDA1: U14.8 (SCK), U15.8 (SCK), U16.8 (SCK), U17.8 (SCK), U18.8 (SCK), U19.8 (SCK), U2.4 (GPIO2), U20.8 (SCK), U21.8 (SCK)
- new net SS: U2.56 (~{QSPI_SS}), U5.1 (~{CS})
- new net XIN: C29.1, U2.20 (XIN), Y1.1
- new net XOUT: R11.2, U2.21 (XOUT)

Commit message: end me
Parts:
- removed C40, C41, C42, C43, C44, C45, C46, C47: 100nf, Capacitor_SMD:C_0402_1005Metric_Pad0.74x0.62mm_HandSolder, symbol Device:C_Small
- removed R18, R22, R26, R27, R30, R32, R38, R39, R40, R41, R42, R43: 2.2k, Resistor_SMD:R_0402_1005Metric_Pad0.72x0.64mm_HandSolder, symbol Device:R_Small
- removed U14, U15, U16, U17, U18, U19, U20, U21: MCP23017, Package_DFN_QFN:QFN-28-1EP_6x6mm_P0.65mm_EP4.25x4.25mm, symbol Interface_Expansion:MCP23017x-x-ML
- added Q1: NMOS, symbol Simulation_SPICE:NMOS
- D3: footprint (none) -> Taranium-libs:USB-C-SMD_20P-P0.50-L6.5-W8.9
- J1, J2: footprint (none) -> Connector_PinSocket_2.54mm:PinSocket_2x20_P2.54mm_Vertical
- R10, R9: value 22 -> 27
Connections:
- net SLEEP: now reaches U2.6 (GPIO4)

Commit message: commit
Parts:
- removed C34, C35, C36, C37, C38, C39: 100nf, Capacitor_SMD:C_0402_1005Metric_Pad0.74x0.62mm_HandSolder, symbol Device:C_Small
- removed Q1: NMOS, symbol Simulation_SPICE:NMOS
- removed R21, R24, R25, R28, R29, R31, R33, R34, R35, R36, R37: 2.2k, Resistor_SMD:R_0402_1005Metric_Pad0.72x0.64mm_HandSolder, symbol Device:R_Small
- removed U10, U11, U12, U13, U8, U9: MCP23017, Package_DFN_QFN:QFN-28-1EP_6x6mm_P0.65mm_EP4.25x4.25mm, symbol Interface_Expansion:MCP23017x-x-ML
- added H1, H2, H3, H4: MountingHole, MountingHole:MountingHole_3.2mm_M3_Pad_Via, symbol Mechanical:MountingHole
- added J10, J9: Conn_01x20_Pin, Connector_PinHeader_2.54mm:PinHeader_1x20_P2.54mm_Vertical, symbol Connector:Conn_01x20_Pin
- added J11: Conn_01x12_Pin, Connector_PinHeader_2.54mm:PinHeader_1x12_P2.54mm_Vertical, symbol Connector:Conn_01x12_Pin
- added J6: +12V, Taranium-libs:5P_Screw_Terminal, symbol Connector:Screw_Terminal_01x05
- added J7: +3V3, Taranium-libs:5P_Screw_Terminal, symbol Connector:Screw_Terminal_01x05
- added J8: GND, Taranium-libs:5P_Screw_Terminal, symbol Connector:Screw_Terminal_01x05
- added R12, R16: 10k, Resistor_SMD:R_01005_0402Metric, symbol Device:R_Small
- added R15: 300, Resistor_SMD:R_01005_0402Metric, symbol Device:R_Small
- added SW2, SW3: SW_Push, Taranium-libs:C720477, symbol Switch:SW_Push
- C11, C12, C13, C14, C15, C16, C17, C29, C30, C4: footprint Capacitor_SMD:C_0201_0603Metric_Pad0.64x0.40mm_HandSolder -> Capacitor_SMD:C_0603_1608Metric_Pad1.08x0.95mm_HandSolder
- D1: footprint Diode_THT:Diode_Bridge_Round_D9.8mm -> Taranium-libs:DIO-BG-TH_KBPC25
- J1: footprint Connector_PinSocket_2.54mm:PinSocket_2x20_P2.54mm_Vertical -> Taranium-libs:240V Power Outlet
- J2: footprint Connector_PinSocket_2.54mm:PinSocket_2x20_P2.54mm_Vertical -> Taranium-libs:USB-C-SMD_20P-P0.50-L6.5-W8.9
- R17: value 2.2k -> 300; footprint Resistor_SMD:R_0402_1005Metric_Pad0.72x0.64mm_HandSolder -> Resistor_SMD:R_01005_0402Metric
Connections:
- net SDA1 is gone; now on net SLEEP: U2.4 (GPIO2)
- net +12V: now also J6.1 (Pin_1), J6.2 (Pin_2), J6.3 (Pin_3), J6.4 (Pin_4), J6.5 (Pin_5)
- net +3V3: now also U7.11 (A0), U7.12 (A1), U7.13 (A2), J7.1 (Pin_1), J7.2 (Pin_2), J7.3 (Pin_3), J7.4 (Pin_4), J7.5 (Pin_5), R12.1, R16.1; no longer R17.1
- net GND: now also U6.29 (EP), U7.29 (EP), J8.1 (Pin_1), J8.2 (Pin_2), J8.3 (Pin_3), J8.4 (Pin_4), J8.5 (Pin_5), SW2.1, SW3.1; no longer U7.12 (A1), U7.13 (A2)
- net SLEEP: no longer U2.6 (GPIO4)
- net at R17.2: now also U7.14 (~{RESET}); no longer U7.11 (A0)
- net at U6.14 (~{RESET}): now also R15.2
- net SCL1: no longer names the net of U2.5 (GPIO3)
- new net: R16.2, R17.1, SW3.2
- new net: R12.2, R15.1, SW2.2
